Commit message: Bugfix/end effector link stl on master (#31)
* Remove reference to EndEffector_Link.stl in URDF

* Removed the EndEffector_Link stl file

File: kortex_description/urdf/JACO3_URDF_V11.urdf (robot description, URDF)
Before this commit: robot JACO3_URDF_V11, 9 links, 8 joints
Links:
- link EndEffector_Link: mass 0 -> None; geometry 
