Commit message: add (somewhat arbitrary) friction and dampening parameters to the gazebo simulation

File: kortex_description/arms/gen3/7dof/urdf/gen3_macro.xacro (robot description, xacro)
@@ -61,4 +61,5 @@
         effort="39"
         velocity="0.8727" />
+      <dynamics damping="0.5" friction="0.5"/>
     </joint>
     <link name="${prefix}half_arm_1_link">
@@ -95,4 +96,5 @@
         xyz="0 0 1" />
       <limit lower="-2.41" upper="2.41" effort="39" velocity="0.8727" />
+      <dynamics damping="0.5" friction="0.5"/>
     </joint>
     <link name="${prefix}half_arm_2_link">
@@ -131,4 +133,5 @@
         effort="39"
         velocity="0.8727" />
+      <dynamics damping="0.5" friction="0.5"/>
     </joint>
     <link name="${prefix}forearm_link">
@@ -165,4 +168,5 @@
         xyz="0 0 1" />
       <limit lower="-2.66" upper="2.66" effort="39" velocity="0.8727" />
+      <dynamics damping="0.5" friction="0.5"/>
     </joint>
     <link name="${prefix}spherical_wrist_1_link">
@@ -201,4 +205,5 @@
         effort="9"
         velocity="0.8727" />
+      <dynamics damping="0.5" friction="0.5"/>
     </joint>
     <link name="${prefix}spherical_wrist_2_link">
@@ -235,4 +240,5 @@
         xyz="0 0 1" />
       <limit lower="-2.23" upper="2.23" effort="9" velocity="0.8727" />
+      <dynamics damping="0.5" friction="0.5"/>
     </joint>
     <link name="${prefix}bracelet_link">
@@ -271,4 +277,5 @@
         effort="9"
         velocity="0.8727" />
+      <dynamics damping="0.5" friction="0.5"/>
     </joint>
     <link name="${prefix}end_effector_link" />

Commit message: reduce friction

File: kortex_description/arms/gen3/7dof/urdf/gen3_macro.xacro (robot description, xacro)
@@ -61,5 +61,5 @@
         effort="39"
         velocity="0.8727" />
-      <dynamics damping="0.5" friction="0.5"/>
+      <dynamics damping="0.5" friction="0.05"/>
     </joint>
     <link name="${prefix}half_arm_1_link">
@@ -96,5 +96,5 @@
         xyz="0 0 1" />
       <limit lower="-2.41" upper="2.41" effort="39" velocity="0.8727" />
-      <dynamics damping="0.5" friction="0.5"/>
+      <dynamics damping="0.5" friction="0.05"/>
     </joint>
     <link name="${prefix}half_arm_2_link">
@@ -133,5 +133,5 @@
         effort="39"
         velocity="0.8727" />
-      <dynamics damping="0.5" friction="0.5"/>
+      <dynamics damping="0.5" friction="0.05"/>
     </joint>
     <link name="${prefix}forearm_link">
@@ -168,5 +168,5 @@
         xyz="0 0 1" />
       <limit lower="-2.66" upper="2.66" effort="39" velocity="0.8727" />
-      <dynamics damping="0.5" friction="0.5"/>
+      <dynamics damping="0.5" friction="0.05"/>
     </joint>
     <link name="${prefix}spherical_wrist_1_link">
@@ -203,7 +203,7 @@
         xyz="0 0 1" />
       <limit
-        effort="9"
-        velocity="0.8727" />
-      <dynamics damping="0.5" friction="0.5"/>
+        effort="50"
+        velocity="0.8727" />
+      <dynamics damping="0.5" friction="0.05"/>
     </joint>
     <link name="${prefix}spherical_wrist_2_link">
@@ -239,6 +239,6 @@
       <axis
         xyz="0 0 1" />
-      <limit lower="-2.23" upper="2.23" effort="9" velocity="0.8727" />
-      <dynamics damping="0.5" friction="0.5"/>
+      <limit lower="-2.23" upper="2.23" effort="50" velocity="0.8727" />
+      <dynamics damping="0.5" friction="0.05"/>
     </joint>
     <link name="${prefix}bracelet_link">
@@ -275,7 +275,7 @@
         xyz="0 0 1" />
       <limit
-        effort="9"
-        velocity="0.8727" />
-      <dynamics damping="0.5" friction="0.5"/>
+        effort="50"
+        velocity="0.8727" />
+      <dynamics damping="0.5" friction="0.05"/>
     </joint>
     <link name="${prefix}end_effector_link" />
